File: FlailDriver.kicad_pcb (KiCad board)
At the start: 2 copper layers, 93 parts, among them J1 PWR, J2 ROUT, J3 LOUT, J4 GAIN_SEL, J6 AudioJack3_SwitchTR, Q2 MMBT3904, Q4 MMBT3904, Q5 MMBT3904, SW1 PWR, SW3 PWR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

Commit message: bak
Parts:
- moved C2 1.52 mm to (164.1, 111.6)
- moved R2 1.52 mm to (164.1, 113.4)
- moved R6 1.52 mm to (164.1, 109.9)
- moved C1 1.40 mm to (160.0, 111.6)
- moved R1 1.40 mm to (160.0, 113.4)
- moved R4 1.40 mm to (160.0, 109.9)
- moved C21 0.38 mm to (47.1, -18.0)
- moved C22 0.38 mm to (56.3, -18.0)
- moved C23 0.38 mm to (51.7, -18.0)
- moved C24 0.38 mm to (60.8, -18.0)
- moved C19 0.25 mm to (56.0, 23.2)
- moved C4 0.25 mm to (53.1, 31.7)
- moved C5 0.25 mm to (54.9, 31.7)
- moved R10 0.25 mm to (51.9, 19.7)
- moved R14 0.25 mm to (56.0, 19.7)
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
Commit message: commit before routing traces
Parts:
- removed Q2, Q4: MMBT3904, Package_TO_SOT_SMD:SOT-23
- removed R20, R23: 100k, Resistor_SMD:R_0603_1608Metric_Pad1.05x0.95mm_HandSolder_SmallRef
- removed RV3: CTRL3, Crossley_Footprints:SMD_TRIM_JLC_Name
- removed RV4: VOL, Crossley_Footprints:SMD_TRIM_JLC_Name
- removed SW6, SW7: SW_Push, HammerheadAudio:JLC_TactileSw_C318884
- removed the U1 at (54.0, 152.4)
- C1, C10, C11, C12, C13, C16, C2, C3, C4, C5, C6, C7, C8, C9: footprint Capacitor_SMD:C_0603_1608Metric_Pad1.05x0.95mm_HandSolder_SmallRef_Top -> Capacitor_SMD:C_0603_1608Metric_Pad1.05x0.95mm_HandSolder_HiddenRef
- C14, C15, C17, C18, C19, C20, C21, C22, C23, C24, C25, C26, C27, C28, C30, C31: footprint Capacitor_SMD:C_0603_1608Metric_Pad1.05x0.95mm_HandSolder_SmallRef -> Capacitor_SMD:C_0603_1608Metric_Pad1.05x0.95mm_HandSolder_HiddenRef
- R1, R10, R11, R12, R13, R14, R15, R17, R18, R19, R2, R21, R22, R25, R26, R3, R4, R5, R6, R8, R9: footprint Resistor_SMD:R_0603_1608Metric_Pad1.05x0.95mm_HandSolder_SmallRef -> Resistor_SMD:R_0603_1608Metric_Pad1.05x0.95mm_HandSolder_HiddenRef
- R7: footprint Resistor_SMD:R_0603_1608Metric_Pad1.05x0.95mm_HandSolder_SmallRef_Top -> Resistor_SMD:R_0603_1608Metric_Pad1.05x0.95mm_HandSolder_HiddenRef
- moved D2 202.2 mm to (46.9, -10.0), turned to 90 degrees
- moved R17 199.4 mm to (47.8, -6.10), turned to 270 degrees
- moved R22 191.6 mm to (56.6, -6.10), turned to 90 degrees
- moved Q5 179.6 mm to (29.2, 19.2)
- moved R19 179.0 mm to (24.6, 19.2), turned to 270 degrees
- moved R21 178.1 mm to (26.4, 19.2), turned to 270 degrees
- moved RV1 121.6 mm to (49.2, 88.9)
- moved H2 118.2 mm to (54.0, 73.0)
- moved RV2 118.2 mm to (58.7, 88.9)
- moved SW4 111.8 mm to (58.7, 98.4), turned to 90 degrees
- moved U1 68.1 mm to (120.7, 91.3), turned to 0 degrees
- moved C7 67.9 mm to (121.5, 86.6)
- moved R8 67.9 mm to (118.0, 86.6)
- moved C6 67.9 mm to (119.8, 86.6)
- moved R12 67.9 mm to (123.3, 86.6)
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Connections:
- D2 pad 2: Net-(D2-Pad2) -> VCC
- R17 pad 1: VCC -> Net-(D2-Pad1)
- R17 pad 2: Net-(D2-Pad2) -> Net-(R17-Pad2)
- R26 pad 2: Net-(R23-Pad1) -> Net-(R17-Pad2)
- U6 pad 2: Net-(R23-Pad1) -> Net-(R17-Pad2)
- U6 pad 3: Net-(R23-Pad1) -> Net-(R17-Pad2)
Routing:
- net VCC: track 0.00 -> 19.8 mm
Other:
- board outline added: 19 x 212.7 mm
- board text added: "GAIN_SELECT"
- board text removed: "GAIN-SELECT"

Commit message: layout progress
Parts:
- added D3: FAULT, LED_SMD:LED_0805_2012Metric_Pad1.15x1.40mm_HandSolder, F.Cu at (33.3, 85.0)
- added D4: FAULT, LED_SMD:LED_0805_2012Metric_Pad1.15x1.40mm_HandSolder, F.Cu at (38.1, 85.0)
- added R16: 2.2k, Resistor_SMD:R_0603_1608Metric_Pad1.05x0.95mm_HandSolder_HiddenRef, F.Cu at (33.0, 87.7)
- added R20: 2.2k, Resistor_SMD:R_0603_1608Metric_Pad1.05x0.95mm_HandSolder_HiddenRef, F.Cu at (37.4, 87.7)
- added RV3: VOL, Crossley_Footprints:SMD_TRIM_JLC, F.Cu at (39.5, 75.7)
- H1, H2, H3, H4: footprint HammerheadAudio:M3_MOUNT_KEEPOUT_2 -> HammerheadAudio:M3_Plated
- RV1, RV2, RV5, RV6: footprint Crossley_Footprints:SMD_TRIM_JLC_Name -> Crossley_Footprints:SMD_TRIM_JLC
- moved C9 45.7 mm to (55.8, -5.84)
- moved C11 45.6 mm to (50.4, -5.84)
- moved C5 5.58 mm to (60.3, 43.3), turned to 0 degrees
- moved C4 5.58 mm to (47.6, 43.3), turned to 0 degrees
- moved RV6 5.48 mm to (60.3, 39.8), turned to 0 degrees
- moved RV5 5.48 mm to (47.6, 39.8), turned to 0 degrees
- moved C14 4.33 mm to (61.1, -9.51)
- moved C10 2.68 mm to (57.5, -5.84)
- moved R22 2.68 mm to (59.3, -5.84)
- moved R10 1.78 mm to (54.0, 16.6)
- moved R14 1.78 mm to (55.8, 16.6)
- moved C19 1.23 mm to (56.0, 36.1)
- moved C12 0.93 mm to (52.2, -5.84)
- moved C15 0.93 mm to (54.0, -5.84)
- moved R17 0.92 mm to (46.9, -5.84)
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Routing:
- net GND: track 0.00 -> 39.2 mm, vias 0 -> 27
- net VCC: track 19.8 -> 49.5 mm
- net GVDD: track 0.00 -> 29.1 mm
- net R-: track 0.00 -> 20.2 mm
- net L+: track 0.00 -> 20.1 mm
- net R+: track 0.00 -> 18.6 mm
- net L-: track 0.00 -> 18.6 mm
- net Net-(J4-Pad1): track 0.00 -> 16.4 mm
- net Net-(J4-Pad2): track 0.00 -> 7.09 mm
- net Net-(C21-Pad1): track 0.00 -> 6.87 mm
- net Net-(C24-Pad2): track 0.00 -> 6.61 mm
- net Net-(J4-Pad6): track 0.00 -> 6.23 mm
- net Net-(J4-Pad4): track 0.00 -> 6.23 mm
- net Net-(R17-Pad2): track 0.00 -> 5.71 mm
- net Net-(C22-Pad1): track 0.00 -> 5.60 mm
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- added copper zone on B.Cu, net GND
- added copper zone on F.Cu, net GND

Commit message: layout progress
Parts:
- added J5: LEFT, HammerheadAudio:EuroJack_MonoSW_THT_NOREF_SmallHoles_NoSilk, F.Cu at (49.0, 52.4)
- D4: value FAULT -> IND
- J2: value ROUT -> LOUT
- J3: value LOUT -> ROUT
- J6: value AudioJack3_SwitchTR -> RIGHT; footprint Connectors:AUDIO-JACK -> HammerheadAudio:EuroJack_MonoSW_THT_NOREF_SmallHoles_NoSilk
- SW3: value PWR -> SW_Push; footprint HammerheadAudio:JLC_SW_SPDT_SMT_C145845 -> HammerheadAudio:JLC_TactileSw_C318884
- U4: footprint MeowWolf_Templates:TEENSY_3.5_3.6_MINIMAL -> MeowWolf_Templates:TEENSY_4.1_MINIMAL_DROP_IN
- moved SW3 137.9 mm to (58.9, 82.5), turned to 270 degrees
- moved R2 136.8 mm to (47.8, 41.5), turned to 90 degrees
- moved C2 134.3 mm to (49.5, 41.5), turned to 270 degrees
- moved U2 131.9 mm to (50.0, 36.5)
- moved R6 131.9 mm to (51.3, 41.5), turned to 270 degrees
- moved R5 131.5 mm to (53.1, 41.5), turned to 90 degrees
- moved C17 125.4 mm to (59.9, 32.6)
- moved R4 124.0 mm to (56.6, 41.5), turned to 270 degrees
- moved C1 123.5 mm to (58.4, 41.5), turned to 270 degrees
- moved R1 123.0 mm to (60.2, 41.5), turned to 90 degrees
- moved R3 120.4 mm to (54.9, 41.5), turned to 90 degrees
- moved R19 113.2 mm to (60.6, 126.5), turned to 180 degrees
- moved R21 110.9 mm to (60.6, 124.7), turned to 180 degrees
- moved Q5 107.3 mm to (60.6, 121.8), turned to 180 degrees
- moved R12 76.6 mm to (49.1, 67.4), turned to 180 degrees
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Connections:
- net BT4 renamed Net-(U4-Pad7)
- net FAULT renamed Net-(U4-Pad3)
- C10 pad 1: LIN- -> RIN-
- C11 pad 1: RIN+ -> LIN+
- C12 pad 1: RIN- -> LIN-
- C9 pad 1: LIN+ -> RIN+
- SW1 pad 1: Net-(SW1-Pad1) -> VCC
- SW1 pad 3: VCC -> Net-(SW1-Pad3)
- SW3 pad 1: Net-(SW3-Pad1) -> GND
- U2 pad 3: Net-(C1-Pad1) -> Net-(C2-Pad1)
- U2 pad 5: Net-(C2-Pad1) -> Net-(RV5-Pad2)
- U2 pad 6: Net-(RV6-Pad3) -> Net-(C11-Pad2)
- U2 pad 7: Net-(RV6-Pad3) -> Net-(C11-Pad2)
- U3 pad 1: Net-(C11-Pad2) -> Net-(RV6-Pad3)
- U3 pad 2: Net-(C11-Pad2) -> Net-(RV6-Pad3)
- U3 pad 3: Net-(RV5-Pad2) -> Net-(C1-Pad1)
- U4 pad 10: Net-(R16-Pad1) -> Net-(R20-Pad2)
- U4 pad 11: Net-(R20-Pad2) -> Net-(R16-Pad1)
- U4 pad 2: UNMUTE -> Net-(U4-Pad2)
- U4 pad 36: Net-(U4-Pad36) -> UNMUTE
- U4 pad 37: CTRL1 -> MUTE_IN
- U4 pad 38: CTRL2 -> CTRL1
- U4 pad 39: CTRL3 -> CTRL2
- U4 pad 4: BT1 -> Net-(U4-Pad4)
- U4 pad 5: BT2 -> BT1
- U4 pad 6: BT3 -> BT2
- U4 pad 8: MUTE_IN -> Net-(U4-Pad8)
- U6 pad 10: LIN+ -> RIN+
- U6 pad 11: LIN- -> RIN-
- U6 pad 4: RIN+ -> LIN+
- U6 pad 5: RIN- -> LIN-
Routing:
- net VCC: track 49.5 -> 293.4 mm
- net Net-(C9-Pad2): track 0.00 -> 46.8 mm
- net AR: track 0.00 -> 21.3 mm
- net Net-(RV6-Pad3): track 0.00 -> 18.8 mm
- net Net-(R20-Pad2): track 0.00 -> 17.1 mm
- net Net-(RV6-Pad2): track 0.00 -> 16.5 mm
- net Net-(R16-Pad1): track 0.00 -> 16.1 mm
- net AL: track 0.00 -> 13.3 mm
- net Net-(J4-Pad1): track 16.4 -> 28.3 mm
- net GVDD: track 29.1 -> 39.9 mm
- net Net-(C2-Pad1): track 0.00 -> 9.28 mm
- net Net-(C1-Pad1): track 0.00 -> 8.96 mm
- net LIN: track 0.00 -> 7.12 mm
- net RIN: track 0.00 -> 7.12 mm
- net Net-(RV5-Pad3): track 0.00 -> 7.12 mm
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Other:
- board text added: "BT1"
- board text added: "BT2"
- board text added: "CTRL1"
- board text added: "CTRL2"
- board text added: "L/MONO"
- board text added: "MUTE"
- board text added: "RIGHT"
- board text added: "VOL"

Commit message: layout finished
Parts:
- J1, J2, J3: footprint HammerheadAudio:Phoenix_Stacked_Marking2_NoRef_Centered_BoardEdge -> HammerheadAudio:Phoenix_Stacked_BackSilk_Centered_BoardEdge
- turned SW3 to 180 degrees
Connections:
- U4 pad 13: Net-(U4-Pad13) -> BT2
- U4 pad 14: Net-(U4-Pad14) -> BT1
- U4 pad 38: CTRL1 -> VOL
- U4 pad 39: CTRL2 -> CTRL1
- U4 pad 40: VOL -> CTRL2
- U4 pad 5: BT1 -> Net-(U4-Pad5)
- U4 pad 6: BT2 -> Net-(U4-Pad6)
Routing:
- net Net-(Q5-Pad3): track 4.90 -> 168.8 mm, vias 0 -> 2
- net DIN: track 0.00 -> 157.2 mm, vias 0 -> 1
- net +3V3: track 0.00 -> 136.3 mm
- net WS: track 0.00 -> 106.8 mm, vias 0 -> 1
- net BCK: track 0.00 -> 98.7 mm, vias 0 -> 1
- net VOL: track 0.00 -> 73.6 mm
- net CTRL1: track 0.00 -> 69.0 mm, vias 0 -> 1
- net CTRL2: track 0.00 -> 63.1 mm, vias 0 -> 1
- net MUTE_IN: track 0.00 -> 61.3 mm
- net +5V: track 2.50 -> 58.8 mm
- net Net-(C11-Pad2): track 0.00 -> 47.0 mm
- net BT1: track 0.00 -> 43.1 mm, vias 0 -> 3
- net BT2: track 0.00 -> 34.5 mm, vias 0 -> 1
- net Net-(D3-Pad2): track 0.00 -> 31.1 mm
- net Net-(D4-Pad2): track 0.00 -> 29.1 mm
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Other:
- board text added: "+ L/MONO -"
- board text added: "+ RIGHT -"
- board text added: "- POWER +"
- board text added: "FUNC"
- board text added: "TRIG"
- board text removed: "BT1"
- board text removed: "BT2"

Commit message: bak
Parts:
- added REF**: JLC_ToolingHole, HammerheadAudio:JLC_ToolingHole, F.Cu at (58.8, -32.4)
- added REF**: JLC_ToolingHole, HammerheadAudio:JLC_ToolingHole, F.Cu at (49.1, -32.4)
- added REF**: JLC_ToolingHole, HammerheadAudio:JLC_ToolingHole, F.Cu at (48.9, 151.1)
- added REF**: JLC_ToolingHole, HammerheadAudio:JLC_ToolingHole, F.Cu at (58.9, 151.1)
Other:
- board text added: "FLAIL DRIVER V1.0 EMMETT PALAIMA HHAUDIO - MAY 2023 JLCJLCJLCJLC"
