File: FlailDriver.kicad_pcb (KiCad board)
At the start: 2 copper layers, 19 x 212.7 mm, 95 parts, among them J1 PWR, J2 LOUT, J3 ROUT, J4 GAIN_SEL, J5 LEFT, J6 RIGHT, Q5 MMBT3904, SW1 PWR, SW3 SW_Push, SW4 SW_Push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

Commit message: newreg
Parts:
- added SW2: SW_DIP_x02, HammerheadAudio:JLC_SMD_DIP_SPSTx2_C40735, F.Cu at (54.0, 81.4)
- U5: value MC7805BDTRKG -> R-78E5.0-1.0; footprint Package_TO_SOT_SMD:TO-263-2 -> HammerheadAudio:TRACO_DCDC; moved to B.Cu
- moved C16 12.1 mm to (60.3, 116.3), turned to 90 degrees
- moved RV3 8.73 mm to (49.0, 89.0)
- moved SW3 8.73 mm to (58.9, 89.0)
- moved RV1 7.94 mm to (49.0, 97.2)
- moved RV2 7.94 mm to (58.9, 97.2)
- moved C13 7.25 mm to (47.6, 116.3), turned to 270 degrees
- moved D3 7.14 mm to (49.0, 103.7)
- moved D4 7.14 mm to (58.9, 103.7)
- moved R16 7.14 mm to (52.8, 108.9)
- moved R20 7.14 mm to (55.1, 108.9)
- moved SW4 7.14 mm to (58.9, 108.9)
- moved SW5 7.14 mm to (49.0, 108.9)
- moved U5 2.37 mm to (54.0, 116.3), turned to 180 degrees
Routing:
- net GND: track 51.6 -> 111.9 mm, vias 74 -> 43
- net RIN: track 7.12 -> 58.5 mm, vias 0 -> 1
- net LIN: track 7.12 -> 51.7 mm, vias 0 -> 1
- net Net-(C16-Pad1): track 40.7 -> 17.7 mm
- net AL: track 12.8 -> 32.6 mm, vias 0 -> 1
- net AR: track 21.0 -> 40.0 mm
- net VCC: track 295.6 -> 304.6 mm
- net VOL: track 73.6 -> 64.8 mm
- net CTRL1: track 71.5 -> 62.9 mm
- net BT1: track 58.3 -> 50.2 mm
- net Net-(R20-Pad2): track 56.1 -> 48.3 mm
- net CTRL2: track 61.2 -> 53.5 mm
- net MUTE_IN: track 61.3 -> 53.7 mm
- net BT2: track 42.1 -> 34.6 mm
- net Net-(R16-Pad1): track 46.4 -> 39.0 mm
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Other:
- board text added: "AUX OUT"
- board text added: "FLAIL DRIVER V1.2 EMMETT PALAIMA HHAUDIO - MAY 2024 JLCJLCJLCJLC"
- board text removed: "FLAIL DRIVER V1.1 EMMETT PALAIMA HHAUDIO - JULY 2023 JLCJLCJLCJLC"

Commit message: bak
Parts:
- U4: footprint MeowWolf_Templates:TEENSY_4.1_MINIMAL_DROP_IN -> MeowWolf_Templates:TEENSY_4.1_MINIMAL_DROP_IN_2
- moved U4 0.79 mm to (54.0, 146.8)
Routing:
- net VOL: track 64.8 -> 65.7 mm
- net WS: track 99.8 -> 99.0 mm
- net +5V: track 45.4 -> 46.2 mm
- net BCK: track 98.6 -> 99.4 mm
- net BT2: track 34.6 -> 35.4 mm
- net MUTE_IN: track 53.7 -> 54.4 mm
- net CTRL1: track 62.9 -> 63.5 mm
- net Net-(R16-Pad1): track 39.0 -> 39.6 mm
- net UNMUTE: track 67.3 -> 67.9 mm
- net BT1: track 50.2 -> 50.8 mm
